File: CAD/LLK.kicad_pcb (KiCad board)
At the start: 2 copper layers, 44.8 x 51.6 mm, 10 parts

Commit message: gerbers
Parts:
- removed kibuzzard-637E6C8C: G***, kibuzzard-637E6C8C
- added G***: BP Logo, BadgePiratesLogos:BPSkull_Distressed_B.SILK, F.Cu at (166.3, 109.8)
- added G***: LOGO, BadgePiratesLogos:BadgePiratesURL_B.SLK, F.Cu at (169.4, 95.8)
- added kibuzzard-639739B8: G***, kibuzzard-639739B8, B.Cu at (140.1, 114.7)
